File: hardware/psithemius/psithemius.sch (KiCad schematic (older format))
At the start: 49 parts, among them J1 Psionic Input, J2 PJ-051AH, J3 7761, J4 AVR-ISP-6, J5 Internal Power, SW1 B3F-4050, SW2 B3F-4050, SW3 B3F-4050, SW4 JS202011AQN, U1 ATtiny84A-PU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

Commit message: added pdfs and jpgs
Parts:
- C11: Manufacturer Würth Elektronik -> Nichicon
- C6: Digi-Key 493-6096-1-ND -> 493-15996-ND; Manufacturer Würth Elektronik -> Nichicon; Mouser Part Number 647-UVR1C221MED1TA -> 647-USR1C221MDD; Mouser/http https://www2.mouser.com/ProductDetail/Nichicon/UVR1C221MED1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 -> https://www2.mouser.com/ProductDetail/Nichicon/USR1C221MDD; Part Number UVR1C221MED1TA -> USR1C221MDD
Changed lines of the file:
@@
 F 1 "220uF/16V" V 8244 2125 30  0000 C CNN
 F 2 "Capacitor_THT:CP_Radial_D8.0mm_P5.00mm" H 8100 2125 50  0001 C CNN
-F 3 "https://www.nichicon.co.jp/english/products/pdfs/e-uvr.pdf" H 8100 2125 50  0001 C CNN
-F 4 "493-6096-1-ND" H 8100 2125 50  0001 C CNN "Digi-Key"
-F 5 "Würth Elektronik" H 8100 2125 50  0001 C CNN "Manufacturer"
-F 6 "UVR1C221MED1TA" H 8100 2125 50  0001 C CNN "Part Number"
+F 3 "http://nichicon-us.com/english/products/pdfs/e-usa_usr.pdf" H 8100 2125 50  0001 C CNN
+F 4 "493-15996-ND" H 8100 2125 50  0001 C CNN "Digi-Key"
+F 5 "Nichicon" H 8100 2125 50  0001 C CNN "Manufacturer"
+F 6 "USR1C221MDD" H 8100 2125 50  0001 C CNN "Part Number"
 F 7 "https://www.digikey.com/product-detail/en/nichicon/UVR1C221MED1TA/493-6096-1-ND/3438470" V 8100 2125 50  0001 C CNN "Digi-Key/http"
-F 8 "647-UVR1C221MED1TA" H 8100 2125 50  0001 C CNN "Mouser Part Number"
-F 9 "https://www2.mouser.com/ProductDetail/Nichicon/UVR1C221MED1TA" H 8100 2125 50  0001 C CNN "Mouser/http"
+F 8 "647-USR1C221MDD" H 8100 2125 50  0001 C CNN "Mouser Part Number"
+F 9 "https://www2.mouser.com/ProductDetail/Nichicon/USR1C221MDD" H 8100 2125 50  0001 C CNN "Mouser/http"
 	1    8100 2125
 	0    -1   -1   0
@@
 F 3 "http://nichicon-us.com/english/products/pdfs/e-usa_usr.pdf" H 2085 3540 50  0001 C CNN
 F 4 "493-15996-ND" H 2085 3540 50  0001 C CNN "Digi-Key"
-F 5 "Würth Elektronik" H 2085 3540 50  0001 C CNN "Manufacturer"
+F 5 "Nichicon" H 2085 3540 50  0001 C CNN "Manufacturer"
 F 6 "USR1C221MDD" H 2085 3540 50  0001 C CNN "Part Number"
 F 7 "https://www.digikey.com/product-detail/en/nichicon/UVR1C221MED1TA/493-6096-1-ND/3438470" V 2085 3540 50  0001 C CNN "Digi-Key/http"
